File: hardware/HS8836A_USBC_hub/HS8836A_USBC_hub.kicad_pcb (KiCad board)
At the start: 2 copper layers, 25 x 84 mm, 18 parts, among them J1 USB_C, J2 USB_A, J3 USB_A, J4 USB_A, J5 USB_A, J6 USB_B, U1 HS8836A

Commit message: swapped dp and dm lines on the controller
Parts:
- J1: value USB_C -> USB_C_Receptacle_USB2.0
- J6: value USB_B -> USB_B_Micro
Connections:
- U1 pad 10: D+ -> D-
- U1 pad 11: D- -> D+
Routing:
- net D-: track 57.9 -> 53.1 mm, vias 3 -> 2
Changed lines of the file:
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@@
         (effects (font (size 0.5 0.5) (thickness 0.075)))
     )
-    (fp_text value "USB_B" (at 0.3 -4.7 90) (layer "F.SilkS")
+    (fp_text value "USB_B_Micro" (at 0.3 -4.7 90) (layer "F.SilkS")
         (effects (font (size 1 1) (thickness 0.15)))
     )
@@
       (net 14 "Net-(U1-REF)") (pinfunction "REF") (pintype "output"))
     (pad "10" smd roundrect (at 3.0875 3.175) (size 1.825 0.65) (layers "F.Cu" "F.Paste" "F.Mask") (roundrect_rratio 0.25)
-      (net 17 "D+") (pinfunction "UM") (pintype "input"))
+      (net 18 "D-") (pinfunction "UM") (pintype "input"))
     (pad "11" smd roundrect (at 3.0875 1.905) (size 1.825 0.65) (layers "F.Cu" "F.Paste" "F.Mask") (roundrect_rratio 0.25)
-      (net 18 "D-") (pinfunction "UP") (pintype "input"))
+      (net 17 "D+") (pinfunction "UP") (pintype "input"))
     (pad "12" smd roundrect (at 3.0875 0.635) (size 1.825 0.65) (layers "F.Cu" "F.Paste" "F.Mask") (roundrect_rratio 0.25)
       (net 1 "Net-(U1-DCP)") (pinfunction "DCP") (pintype "output"))
@@
         (effects (font (size 0.5 0.5) (thickness 0.075)))
     )
-    (fp_text value "USB_C" (at -0.2 1.9 90) (layer "F.SilkS")
+    (fp_text value "USB_C_Receptacle_USB2.0" (at -0.2 1.9 90) (layer "F.SilkS")
         (effects (font (size 1 1) (thickness 0.15)))
     )
@@
   (segment (start 147.8 76.45) (end 156.725 76.45) (width 0.25) (layer "F.Cu") (net 16))
   (segment (start 156.725 76.45) (end 156.975 76.7) (width 0.25) (layer "F.Cu") (net 16))
+  (segment (start 147.828 100.24) (end 149.823 100.24) (width 0.2) (layer "F.Cu") (net 17))
+  (segment (start 146.214 100.24) (end 145.5356 99.5616) (width 0.2) (layer "F.Cu") (net 17))
+  (segment (start 147.828 100.24) (end 146.214 100.24) (width 0.2) (layer "F.Cu") (net 17))
   (segment (start 149.1594 78.45) (end 147.757 78.45) (width 0.2) (layer "F.Cu") (net 17))
-  (segment (start 145.9484 99.3648) (end 145.5356 98.952) (width 0.2) (layer "F.Cu") (net 17))
   (segment (start 149.352 77.6732) (end 149.352 78.2574) (width 0.2) (layer "F.Cu") (net 17))
-  (segment (start 147.828 101.51) (end 149.5414 101.51) (width 0.2) (layer "F.Cu") (net 17))
-  (segment (start 147.828 101.51) (end 146.8998 101.51) (width 0.2) (layer "F.Cu") (net 17))
+  (segment (start 145.5356 99.5616) (end 145.5356 98.952) (width 0.2) (layer "F.Cu") (net 17))
   (segment (start 145.9082 78.45) (end 147.757 78.45) (width 0.2) (layer "F.Cu") (net 17))
-  (segment (start 145.9484 100.5586) (end 145.9484 99.3648) (width 0.2) (layer "F.Cu") (net 17))
   (segment (start 145.5356 88.243214) (end 145.0361 87.743714) (width 0.2) (layer "F.Cu") (net 17))
   (segment (start 147.757 77.45) (end 149.1288 77.45) (width 0.2) (layer "F.Cu") (net 17))
   (segment (start 144.175 120.4) (end 146.6 120.4) (width 0.2) (layer "F.Cu") (net 17))
-  (segment (start 147.41 101.51) (end 147.01 101.51) (width 0.2) (layer "F.Cu") (net 17))
   (segment (start 149.352 78.2574) (end 149.1594 78.45) (width 0.2) (layer "F.Cu") (net 17))
-  (segment (start 147.4 101.52) (end 147.41 101.51) (width 0.2) (layer "F.Cu") (net 17))
   (segment (start 149.1288 77.45) (end 149.352 77.6732) (width 0.2) (layer "F.Cu") (net 17))
-  (segment (start 149.5414 101.51) (end 149.8092 101.7778) (width 0.2) (layer "F.Cu") (net 17))
   (segment (start 145.0361 79.3221) (end 145.9082 78.45) (width 0.2) (layer "F.Cu") (net 17))
   (segment (start 146.6 120.4) (end 147.9 119.1) (width 0.2) (layer "F.Cu") (net 17))
+  (segment (start 149.823 100.24) (end 149.86 100.203) (width 0.2) (layer "F.Cu") (net 17))
   (segment (start 145.0361 87.743714) (end 145.0361 79.3221) (width 0.2) (layer "F.Cu") (net 17))
   (segment (start 145.5356 98.952) (end 145.5356 88.243214) (width 0.2) (layer "F.Cu") (net 17))
-  (segment (start 146.8998 101.51) (end 145.9484 100.5586) (width 0.2) (layer "F.Cu") (net 17))
-  (via (at 149.8092 101.7778) (size 0.8) (drill 0.4) (layers "F.Cu" "B.Cu") (net 17))
+  (via (at 149.86 100.203) (size 0.8) (drill 0.4) (layers "F.Cu" "B.Cu") (net 17))
   (via (at 147.9 119.1) (size 0.8) (drill 0.4) (layers "F.Cu" "B.Cu") (net 17))
-  (segment (start 147.1 102.6922) (end 147.1 117.6) (width 0.2) (layer "B.Cu") (net 17))
-  (segment (start 148.0144 101.7778) (end 147.1 102.6922) (width 0.2) (layer "B.Cu") (net 17))
+  (segment (start 147.1 101.439) (end 147.1 117.6) (width 0.2) (layer "B.Cu") (net 17))
+  (segment (start 148.336 100.203) (end 147.1 101.439) (width 0.2) (layer "B.Cu") (net 17))
   (segment (start 147.9 118.4) (end 147.9 119.1) (width 0.2) (layer "B.Cu") (net 17))
-  (segment (start 149.8092 101.7778) (end 148.0144 101.7778) (width 0.2) (layer "B.Cu") (net 17))
+  (segment (start 149.86 100.203) (end 148.336 100.203) (width 0.2) (layer "B.Cu") (net 17))
   (segment (start 147.1 117.6) (end 147.9 118.4) (width 0.2) (layer "B.Cu") (net 17))
   (segment (start 146.220914 77.5716) (end 144.6361 79.156415) (width 0.2) (layer "F.Cu") (net 18))
@@
   (segment (start 146.4564 77.1398) (end 146.4564 77.5716) (width 0.2) (layer "F.Cu") (net 18))
   (segment (start 145.1356 100.203) (end 145.1356 88.4089) (width 0.2) (layer "F.Cu") (net 18))
+  (segment (start 147.828 101.51) (end 146.4426 101.51) (width 0.2) (layer "F.Cu") (net 18))
+  (segment (start 147.41 101.51) (end 147.01 101.51) (width 0.2) (layer "F.Cu") (net 18))
+  (segment (start 147.4 101.52) (end 147.41 101.51) (width 0.2) (layer "F.Cu") (net 18))
   (segment (start 146.6462 76.95) (end 146.4564 77.1398) (width 0.2) (layer "F.Cu") (net 18))
   (segment (start 146.4564 77.5716) (end 146.4564 77.6986) (width 0.2) (layer "F.Cu") (net 18))
-  (segment (start 149.823 100.24) (end 149.8346 100.2284) (width 0.2) (layer "F.Cu") (net 18))
   (segment (start 145.1356 88.4089) (end 144.6361 87.9094) (width 0.2) (layer "F.Cu") (net 18))
   (segment (start 146.4564 77.5716) (end 146.220914 77.5716) (width 0.2) (layer "F.Cu") (net 18))
+  (segment (start 146.4426 101.51) (end 145.1356 100.203) (width 0.2) (layer "F.Cu") (net 18))
   (segment (start 146.7078 77.95) (end 146.4564 77.6986) (width 0.2) (layer "F.Cu") (net 18))
-  (segment (start 147.828 100.24) (end 149.823 100.24) (width 0.2) (layer "F.Cu") (net 18))
   (via (at 146.7 119) (size 0.8) (drill 0.4) (layers "F.Cu" "B.Cu") (net 18))
-  (via (at 149.8346 100.2284) (size 0.8) (drill 0.4) (layers "F.Cu" "B.Cu") (net 18))
   (via (at 145.1356 100.203) (size 0.8) (drill 0.4) (layers "F.Cu" "B.Cu") (net 18))
-  (segment (start 149.8346 100.2284) (end 147.8534 100.2284) (width 0.2) (layer "B.Cu") (net 18))
-  (segment (start 146.7 101.3818) (end 146.7 119) (width 0.2) (layer "B.Cu") (net 18))
-  (segment (start 149.8346 100.2284) (end 145.161 100.2284) (width 0.2) (layer "B.Cu") (net 18))
-  (segment (start 147.8534 100.2284) (end 146.7 101.3818) (width 0.2) (layer "B.Cu") (net 18))
+  (segment (start 145.161 100.203) (end 146.7 101.742) (width 0.2) (layer "B.Cu") (net 18))
+  (segment (start 146.7 101.742) (end 146.7 119) (width 0.2) (layer "B.Cu") (net 18))
+  (segment (start 145.1356 100.203) (end 145.161 100.203) (width 0.2) (layer "B.Cu") (net 18))
   (segment (start 145.161 100.2284) (end 145.1356 100.203) (width 0.2) (layer "B.Cu") (net 18))
   (segment (start 147.8 79.45) (end 156.725 79.45) (width 0.25) (layer "F.Cu") (net 20))

Commit message: Updated Gerbers and images
Other:
- board text added: "EZER LONGINUS APR 2024"
- board text removed: "EZER LONGINUS MAR 2024"
